Commit message: update z1 urdf (EE part)

File: z1.urdf (robot description, URDF)
Before this commit: robot z1_description, 8 links, 7 joints
Links:
- added link gripperMover, mass 0.27621302; collision mesh filename=package://example-robot-data/robots/z1_description/meshes/c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 scale=1 1 1; visual mesh filename=package://example-robot-data/robots/z1_description/meshes/v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 scale=1 1 1
- added link gripperStator, mass 0.52603655; collision mesh filename=package://example-robot-data/robots/z1_description/meshes/c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 scale=1 1 1; visual mesh filename=package://example-robot-data/robots/z1_description/meshes/v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 scale=1 1 1
- link link00: geometry collision cylinder length=0.051 radius=0.0325; visual mesh filename=package://example-robot-data/robots/z1_description/meshes/v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 scale=1 1 1
- link link01: geometry visual mesh filename=package://example-robot-data/robots/z1_description/meshes/v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 scale=1 1 1
- link link02: geometry collision cylinder length=0.051 radius=0.0325; collision cylinder length=0.102 radius=0.0325
- link link03: geometry collision cylinder length=0.059 radius=0.0325; collision cylinder length=0.116 radius=0.02
- link link04: geometry collision cylinder length=0.067 radius=0.0325; visual mesh filename=package://example-robot-data/robots/z1_description/meshes/v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 scale=1 1 1
- link link05: geometry visual mesh filename=package://example-robot-data/robots/z1_description/meshes/v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 scale=1 1 1
- link link06: geometry collision cylinder length=0.051 radius=0.0325; visual mesh filename=package://example-robot-data/robots/z1_description/meshes/v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 scale=1 1 1
Joints:
- added joint gripperStator: type fixed, parent link06, child gripperStator, origin xyz=0.051 0.0 0.0 rpy=0 0 0
- added joint jointGripper: type revolute, parent gripperStator, child gripperMover, origin xyz=0.049 0.0 0 rpy=0 0 0, axis 0 1 0, limit lower=-1.5707 upper=0.0 effort=30. velocity=3.1415
